File: clumsyMIDI.sch (KiCad schematic (older format))
At the start: 21 parts, among them J2 MIDI Out Jack, J3 MIDI In Jack, J4 MIDI Thru Jack, P1 Conn_02x20_Odd_Even, U1 74HCT14, U2 H11L1M

Commit message: fixed the MIDI connector symbols in the schematic (no PCB change)
Parts:
- J2, J3, J4: symbol Connector:DIN-5 -> Connector:DIN-5_180degree
Connections:
- wire segments 156 -> 151
Changed lines of the file:
@@
 $EndComp
-Wire Wire Line
-	6675 1425 6675 1725
 Wire Wire Line
 	6675 1725 6525 1725
 Wire Wire Line
 	6850 1800 6850 1925
-Wire Wire Line
-	6850 1500 6850 1425
 $Comp
 L power:GND #PWR011
@@
 	5175 2200 5175 2075
 Connection ~ 5175 2075
-NoConn ~ 8200 2125
-NoConn ~ 8500 1925
-NoConn ~ 8500 1725
-Wire Wire Line
-	7675 1725 7675 1425
-Wire Wire Line
-	7900 1725 7675 1725
-Wire Wire Line
-	7575 1925 7900 1925
 $Comp
 L Device:R R4
@@
 	0    1    1    0
 $EndComp
-$Comp
-L Connector:DIN-5 J3
-U 1 1 5F99CA21
-P 8200 1825
-F 0 "J3" H 8200 1458 50  0000 C CNN
-F 1 "MIDI In Jack" H 8200 1549 50  0000 C CNN
-F 2 "clumsyMIDI:MultiDIN5" H 8200 1825 50  0001 C CNN
-F 3 "http://www.mouser.com/ds/2/18/40_c091_abd_e-75918.pdf" H 8200 1825 50  0001 C CNN
-	1    8200 1825
-	-1   0    0    1
-$EndComp
 Wire Wire Line
 	7275 1925 6850 1925
-Wire Wire Line
-	6850 1425 7675 1425
-Wire Wire Line
-	6675 1425 6850 1425
-Connection ~ 6850 1425
 Wire Wire Line
 	6850 1925 6525 1925
@@
 Connection ~ 5175 1825
 $Comp
-L Connector:DIN-5 J2
+L Connector:DIN-5_180degree J2
 U 1 1 5FBFBE67
-P 5425 6275
-F 0 "J2" H 5425 5908 50  0000 C CNN
-F 1 "MIDI Out Jack" H 5425 5999 50  0000 C CNN
-F 2 "clumsyMIDI:MultiDIN5" H 5425 6275 50  0001 C CNN
-F 3 "http://www.mouser.com/ds/2/18/40_c091_abd_e-75918.pdf" H 5425 6275 50  0001 C CNN
-	1    5425 6275
+P 5350 6200
+F 0 "J2" H 5350 5833 50  0000 C CNN
+F 1 "MIDI Out Jack" H 5350 5924 50  0000 C CNN
+F 2 "clumsyMIDI:MultiDIN5" H 5350 6200 50  0001 C CNN
+F 3 "" H 5350 6200 50  0001 C CNN
+	1    5350 6200
 	-1   0    0    1
 $EndComp
 $Comp
-L Connector:DIN-5 J4
+L Connector:DIN-5_180degree J4
 U 1 1 5FBFCA41
 P 10175 2050
@@
 F 1 "MIDI Thru Jack" H 10175 1774 50  0000 C CNN
 F 2 "Connector_PinHeader_2.54mm:PinHeader_1x05_P2.54mm_Vertical" H 10175 2050 50  0001 C CNN
-F 3 "http://www.mouser.com/ds/2/18/40_c091_abd_e-75918.pdf" H 10175 2050 50  0001 C CNN
+F 3 "" H 10175 2050 50  0001 C CNN
 	1    10175 2050
 	-1   0    0    1
@@
 L power:+5V #PWR019
 U 1 1 5FC2F26A
-P 9775 2550
-F 0 "#PWR019" H 9775 2400 50  0001 C CNN
-F 1 "+5V" H 9775 2690 50  0000 C CNN
-F 2 "" H 9775 2550 50  0000 C CNN
-F 3 "" H 9775 2550 50  0000 C CNN
-	1    9775 2550
+P 10625 2550
+F 0 "#PWR019" H 10625 2400 50  0001 C CNN
+F 1 "+5V" H 10625 2690 50  0000 C CNN
+F 2 "" H 10625 2550 50  0000 C CNN
+F 3 "" H 10625 2550 50  0000 C CNN
+	1    10625 2550
 	-1   0    0    1
 $EndComp
@@
 L Device:R R5
 U 1 1 5FC30A93
-P 9775 2350
-F 0 "R5" H 9705 2304 50  0000 R CNN
-F 1 "220R" H 9705 2395 50  0000 R CNN
-F 2 "Resistor_THT:R_Axial_DIN0207_L6.3mm_D2.5mm_P7.62mm_Horizontal" V 9705 2350 50  0001 C CNN
-F 3 "~" H 9775 2350 50  0001 C CNN
-	1    9775 2350
+P 10625 2350
+F 0 "R5" H 10555 2304 50  0000 R CNN
+F 1 "220R" H 10555 2395 50  0000 R CNN
+F 2 "Resistor_THT:R_Axial_DIN0207_L6.3mm_D2.5mm_P7.62mm_Horizontal" V 10555 2350 50  0001 C CNN
+F 3 "~" H 10625 2350 50  0001 C CNN
+	1    10625 2350
 	-1   0    0    1
 $EndComp
 Wire Wire Line
-	9775 2200 9775 2150
-Wire Wire Line
-	9775 2550 9775 2500
-Wire Wire Line
-	9875 2150 9775 2150
+	10625 2550 10625 2500
 $Comp
 L power:GND #PWR021
 U 1 1 5FC5484B
-P 10575 2525
-F 0 "#PWR021" H 10575 2275 50  0001 C CNN
-F 1 "GND" H 10580 2352 50  0000 C CNN
-F 2 "" H 10575 2525 50  0001 C CNN
-F 3 "" H 10575 2525 50  0001 C CNN
-	1    10575 2525
-	1    0    0    -1
-$EndComp
-Wire Wire Line
-	10575 2525 10575 2150
-Wire Wire Line
-	10575 2150 10475 2150
-NoConn ~ 10475 1950
-NoConn ~ 10175 2350
+P 10175 2525
+F 0 "#PWR021" H 10175 2275 50  0001 C CNN
+F 1 "GND" H 10180 2352 50  0000 C CNN
+F 2 "" H 10175 2525 50  0001 C CNN
+F 3 "" H 10175 2525 50  0001 C CNN
+	1    10175 2525
+	1    0    0    -1
+$EndComp
+NoConn ~ 10475 2050
 Wire Wire Line
 	10700 1125 10775 1125
@@
 Wire Wire Line
 	10775 1525 9700 1525
-Wire Wire Line
-	9700 1525 9700 1950
-Wire Wire Line
-	9700 1950 9875 1950
 Wire Wire Line
 	9100 2150 9100 1875
@@
 L power:+5V #PWR010
 U 1 1 5FD00C6D
-P 5025 6775
-F 0 "#PWR010" H 5025 6625 50  0001 C CNN
-F 1 "+5V" H 5025 6915 50  0000 C CNN
-F 2 "" H 5025 6775 50  0000 C CNN
-F 3 "" H 5025 6775 50  0000 C CNN
-	1    5025 6775
+P 5650 6700
+F 0 "#PWR010" H 5650 6550 50  0001 C CNN
+F 1 "+5V" H 5650 6840 50  0000 C CNN
+F 2 "" H 5650 6700 50  0000 C CNN
+F 3 "" H 5650 6700 50  0000 C CNN
+	1    5650 6700
 	-1   0    0    1
 $EndComp
@@
 L Device:R R2
 U 1 1 5FD00C73
-P 5025 6575
-F 0 "R2" H 4955 6529 50  0000 R CNN
-F 1 "220R" H 4955 6620 50  0000 R CNN
-F 2 "Resistor_THT:R_Axial_DIN0207_L6.3mm_D2.5mm_P7.62mm_Horizontal" V 4955 6575 50  0001 C CNN
-F 3 "~" H 5025 6575 50  0001 C CNN
-	1    5025 6575
+P 5650 6500
+F 0 "R2" H 5580 6454 50  0000 R CNN
+F 1 "220R" H 5580 6545 50  0000 R CNN
+F 2 "Resistor_THT:R_Axial_DIN0207_L6.3mm_D2.5mm_P7.62mm_Horizontal" V 5580 6500 50  0001 C CNN
+F 3 "~" H 5650 6500 50  0001 C CNN
+	1    5650 6500
 	-1   0    0    1
 $EndComp
 Wire Wire Line
-	5025 6425 5025 6375
-Wire Wire Line
-	5025 6775 5025 6725
-Wire Wire Line
-	5125 6375 5025 6375
+	5650 6350 5650 6300
+Wire Wire Line
+	5650 6700 5650 6650
 $Comp
 L power:GND #PWR012
 U 1 1 5FD12B0A
-P 5825 6750
-F 0 "#PWR012" H 5825 6500 50  0001 C CNN
-F 1 "GND" H 5830 6577 50  0000 C CNN
-F 2 "" H 5825 6750 50  0001 C CNN
-F 3 "" H 5825 6750 50  0001 C CNN
-	1    5825 6750
-	1    0    0    -1
-$EndComp
-Wire Wire Line
-	5825 6750 5825 6375
-Wire Wire Line
-	5825 6375 5725 6375
+P 5350 6675
+F 0 "#PWR012" H 5350 6425 50  0001 C CNN
+F 1 "GND" H 5355 6502 50  0000 C CNN
+F 2 "" H 5350 6675 50  0001 C CNN
+F 3 "" H 5350 6675 50  0001 C CNN
+	1    5350 6675
+	1    0    0    -1
+$EndComp
 Text GLabel 3000 6850 0    50   Input ~ 0
 TX_TTL
@@
 	4775 6850 4775 6625
 Wire Wire Line
-	4775 6325 4775 6175
-Wire Wire Line
-	4775 6175 5125 6175
-Wire Wire Line
 	3725 6850 3850 6850
 Wire Wire Line
@@
 	9850 5550 9650 5550
 Connection ~ 9650 5550
-NoConn ~ 5725 6175
-NoConn ~ 5425 6575
+NoConn ~ 5650 6200
 NoConn ~ 6650 100
+Wire Wire Line
+	4775 6325 4775 6300
+Wire Wire Line
+	4775 6300 5050 6300
+NoConn ~ 5050 6200
+Wire Wire Line
+	5350 6500 5350 6675
+Wire Wire Line
+	10625 2200 10625 2150
+Wire Wire Line
+	10625 2150 10475 2150
+NoConn ~ 9875 2050
+Wire Wire Line
+	9700 2150 9875 2150
+Wire Wire Line
+	9700 1525 9700 2150
+Wire Wire Line
+	10175 2525 10175 2350
+$Comp
+L Connector:DIN-5_180degree J3
+U 1 1 5F99CA21
+P 8075 1625
+F 0 "J3" H 8075 1258 50  0000 C CNN
+F 1 "MIDI In Jack" H 8075 1349 50  0000 C CNN
+F 2 "clumsyMIDI:MultiDIN5" H 8075 1625 50  0001 C CNN
+F 3 "" H 8075 1625 50  0001 C CNN
+	1    8075 1625
+	0    -1   -1   0
+$EndComp
+Wire Wire Line
+	7575 1925 7975 1925
+Wire Wire Line
+	7975 1325 6850 1325
+Wire Wire Line
+	6675 1325 6675 1725
+Wire Wire Line
+	6850 1325 6850 1500
+Connection ~ 6850 1325
+Wire Wire Line
+	6850 1325 6675 1325
+NoConn ~ 7775 1625
+NoConn ~ 8075 1325
+NoConn ~ 8075 1925
 $EndSCHEMATC
